File: kicad/pathfinder.kicad_pcb (KiCad board)
At the start: 2 copper layers, 73 x 42 mm, 15 parts, among them SW1 SW_Push, SW2 SW_Push, SW3 SW_Push, SW4 SW_Push, U1 XIAO-RP2040-DIP

Commit message: routing
Routing:
- net GND: track 1.86 -> 154.5 mm
- net led4: track 0.00 -> 49.4 mm
- net led5: track 1.50 -> 48.4 mm
- net led2: track 0.00 -> 43.2 mm
- net led1: track 0.00 -> 42.1 mm
- net b4: track 0.84 -> 39.0 mm
- net b2: track 0.00 -> 29.8 mm
- net b3: track 0.00 -> 21.7 mm
- net b1: track 0.00 -> 18.1 mm
- net Net-(D1-PadA): track 0.44 -> 8.88 mm
- net Net-(D3-PadA): track 0.00 -> 7.69 mm
- net Net-(D5-PadA): track 0.00 -> 7.42 mm
- net Net-(D2-PadA): track 0.00 -> 6.77 mm
- net Net-(D4-PadA): track 0.36 -> 4.39 mm
